File: 5v-power.sch (EAGLE design)
At the start: 29 parts, among them IC1 LM2576, J1 Bypass, J2 En, J3 12v, J4 5V Out, J5 LEN EN, Q1 SI4532ADY

Commit message: power pole in and out now added
Parts:
- added J6, J7: POWERPOLE_POWER10AWG, powerpoles:POWERPOLE_POWER10AWG
Connections:
- net 5V: now also J6.V+
- net GND: now also J6.GND, J7.GND
- net N$1: now also J7.V+
Changed lines of the file:
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@@
 <part name="FRAME1" library="frames" deviceset="A4L-LOC" device=""/>
 <part name="J3" library="farnell-parts" deviceset="2-PIN-MOLEX" device="" value="12v"/>
+<part name="J6" library="powerpoles" deviceset="POWERPOLE_POWER" device="10AWG"/>
+<part name="J7" library="powerpoles" deviceset="POWERPOLE_POWER" device="10AWG"/>
 </parts>
 <sheets>
@@
 <attribute name="VALUE" x="78.74" y="117.475" size="1.778" layer="96"/>
 </instance>
+<instance part="J6" gate="G$1" x="200.66" y="76.2"/>
+<instance part="J7" gate="G$1" x="76.2" y="129.54" rot="MR0"/>
 </instances>
 <busses>
@@
 <wire x1="190.5" y1="38.1" x2="190.5" y2="58.42" width="0.1524" layer="91"/>
 <junction x="190.5" y="58.42"/>
+<pinref part="J6" gate="G$1" pin="GND"/>
+<wire x1="190.5" y1="71.12" x2="190.5" y2="58.42" width="0.1524" layer="91"/>
 </segment>
 <segment>
@@
 <pinref part="C6" gate="G$1" pin="-"/>
 <pinref part="J3" gate="G$1" pin="1"/>
-<wire x1="109.22" y1="106.68" x2="86.36" y2="106.68" width="0.1524" layer="91"/>
+<wire x1="109.22" y1="106.68" x2="88.9" y2="106.68" width="0.1524" layer="91"/>
+<wire x1="88.9" y1="106.68" x2="86.36" y2="106.68" width="0.1524" layer="91"/>
 <wire x1="86.36" y1="106.68" x2="86.36" y2="111.76" width="0.1524" layer="91"/>
 <junction x="109.22" y="106.68"/>
+<pinref part="J7" gate="G$1" pin="GND"/>
+<wire x1="86.36" y1="124.46" x2="88.9" y2="124.46" width="0.1524" layer="91"/>
+<wire x1="88.9" y1="124.46" x2="88.9" y2="106.68" width="0.1524" layer="91"/>
+<junction x="88.9" y="106.68"/>
 </segment>
 </net>
@@
 <segment>
 <wire x1="157.48" y1="60.96" x2="167.64" y2="60.96" width="0.1524" layer="91"/>
-<wire x1="167.64" y1="60.96" x2="193.04" y2="60.96" width="0.1524" layer="91"/>
+<wire x1="167.64" y1="60.96" x2="185.42" y2="60.96" width="0.1524" layer="91"/>
+<wire x1="185.42" y1="60.96" x2="193.04" y2="60.96" width="0.1524" layer="91"/>
 <wire x1="193.04" y1="60.96" x2="195.58" y2="60.96" width="0.1524" layer="91"/>
 <wire x1="149.86" y1="60.96" x2="157.48" y2="60.96" width="0.1524" layer="91"/>
@@
 <wire x1="193.04" y1="45.72" x2="193.04" y2="60.96" width="0.1524" layer="91"/>
 <junction x="193.04" y="60.96"/>
+<pinref part="J6" gate="G$1" pin="V+"/>
+<wire x1="190.5" y1="81.28" x2="185.42" y2="81.28" width="0.1524" layer="91"/>
+<wire x1="185.42" y1="81.28" x2="185.42" y2="60.96" width="0.1524" layer="91"/>
+<junction x="185.42" y="60.96"/>
 </segment>
 <segment>
@@
 <pinref part="R4" gate="G$1" pin="2"/>
 <pinref part="J2" gate="G$1" pin="2"/>
+<junction x="38.1" y="71.12"/>
 <wire x1="20.32" y1="71.12" x2="38.1" y2="71.12" width="0.1524" layer="91"/>
-<junction x="38.1" y="71.12"/>
 </segment>
 </net>
@@
 <pinref part="D1" gate="G$1" pin="A"/>
 <wire x1="86.36" y1="114.3" x2="91.44" y2="114.3" width="0.1524" layer="91"/>
-</segment>
-</net>
+<pinref part="J7" gate="G$1" pin="V+"/>
+<wire x1="86.36" y1="134.62" x2="91.44" y2="134.62" width="0.1524" layer="91"/>
+<wire x1="91.44" y1="134.62" x2="91.44" y2="114.3" width="0.1524" layer="91"/>
+<junction x="91.44" y="114.3"/>
+</segment>
+</net>
