File: 5v-low-power.brd (EAGLE design)
At the start: 68.6 x 40.3 mm, 34 parts, among them J1 Bypass, J2 En, J3 12v, J4 5V Out, J5 LED EN, J6 POWERPOLE_POWER25A, J7 POWERPOLE_POWER25A, Q1 SI4532ADY, U1 LT1934ES6TRMPBF

Commit message: uses a4 frame and smaller ground plane area to make printing better
Changed lines of the file:
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@@
 <contactref element="J7" pad="BLACK"/>
 <polygon width="0.6096" layer="16">
-<vertex x="-8.89" y="120.015"/>
-<vertex x="172.72" y="120.015"/>
-<vertex x="172.72" y="-29.845"/>
-<vertex x="-8.89" y="-29.845"/>
+<vertex x="-9.525" y="55.245"/>
+<vertex x="86.36" y="51.435"/>
+<vertex x="77.47" y="-12.065"/>
+<vertex x="-6.35" y="-11.43"/>
 </polygon>
 <polygon width="0.6096" layer="1">
-<vertex x="-3.81" y="113.665"/>
-<vertex x="167.64" y="113.665"/>
-<vertex x="167.64" y="-22.225"/>
-<vertex x="-3.81" y="-22.225"/>
+<vertex x="-3.81" y="45.085"/>
+<vertex x="80.645" y="44.45"/>
+<vertex x="72.39" y="-6.985"/>
+<vertex x="-3.175" y="-8.255"/>
 </polygon>
 <contactref element="C19" pad="2"/>
